Commit message: Small fix in arms URDF

File: hros5_description/urdf/modules/arms.xacro (robot description, xacro)
@@ -12,5 +12,5 @@
 			<xacro:visuals_collisions_shoulder side="${side}" reflect="${reflect}"/>
 		</link>
-		<joint name="${side}ShoulderRoll" type="revolute">
+		<!-- <joint name="${side}ShoulderRoll" type="revolute">
 			<parent link="${side}Shoulder"/>
 			<child link="${side}UpperArm"/>
@@ -18,5 +18,5 @@
 			<axis xyz="1 0 0"/>
 			<limit lower="${reflect*-2.35619449}" upper="${reflect*1.30899694}" effort="10" velocity="2"/>
-		</joint>
+		</joint> -->
 		<link name="${side}UpperArm">
 			<xacro:visuals_collisions_upper_arm side="${side}" reflect="${reflect}"/>
@@ -35,3 +35,17 @@
 	<xacro:arms_links_joints reflect="1" side="L"/>
 	<xacro:arms_links_joints reflect="-1" side="R"/>
+	<joint name="LShoulderRoll" type="revolute">
+		<parent link="LShoulder"/>
+		<child link="LUpperArm"/>
+		<origin xyz="0.002 0.03 -0.03" rpy="0.174532925 0 0"/>
+		<axis xyz="1 0 0"/>
+		<limit lower="-2.35619449" upper="1.30899694" effort="10" velocity="2"/>
+	</joint>
+	<joint name="RShoulderRoll" type="revolute">
+		<parent link="RShoulder"/>
+		<child link="RUpperArm"/>
+		<origin xyz="0.002 -0.03 -0.03" rpy="-0.174532925 0 0"/>
+		<axis xyz="1 0 0"/>
+		<limit lower="-1.30899694" upper="2.35619449" effort="10" velocity="2"/>
+	</joint>
 </robot>

Commit message: Added proper limits to joint according to Dynamixel manuals

File: hros5_description/urdf/modules/arms.xacro (robot description, xacro)
@@ -2,5 +2,5 @@
 <robot xmlns:xacro="http://www.ros.org/wiki/xacro">
 	<xacro:macro name="arms_links_joints" params="side reflect">
-		<joint name="${side}ShoulderPitch" type="continuous">
+		<joint name="${side}ShoulderPitch" type="revolute">
 			<parent link="base_link"/>
 			<child link="${side}Shoulder"/>
@@ -8,4 +8,5 @@
 			<origin xyz="0.003 ${reflect*0.0675} 0.084" rpy="0 0 0"/>
 			<axis xyz="0 1 0"/>
+			<limit lower="-3.14159265" upper="3.14159265" effort="6.0" velocity="6.597344565"/>
 		</joint>
 		<link name="${side}Shoulder">
@@ -17,5 +18,5 @@
 			<origin xyz="0.002 ${reflect*0.03} -0.03" rpy="${reflect*0.174532925} 0 0"/>
 			<axis xyz="1 0 0"/>
-			<limit lower="${reflect*-2.35619449}" upper="${reflect*1.30899694}" effort="10" velocity="2"/>
+			<limit lower="${reflect*-2.35619449}" upper="${reflect*1.30899694}" effort="6.0" velocity="6.597344565"/>
 		</joint> -->
 		<link name="${side}UpperArm">
@@ -27,5 +28,5 @@
 			<origin xyz="0.03 ${reflect*-0.0015} -0.085" rpy="0 0 0"/>
 			<axis xyz="0 1 0"/>
-			<limit lower="${reflect*-1.22173048}" upper="${reflect*1.65806279}" effort="10" velocity="2"/>
+			<limit lower="${reflect*-1.22173048}" upper="${reflect*1.65806279}" effort="6.0" velocity="6.597344565"/>
 		</joint>
 		<link name="${side}LowerArm">
@@ -40,5 +41,5 @@
 		<origin xyz="0.002 0.03 -0.03" rpy="0.174532925 0 0"/>
 		<axis xyz="1 0 0"/>
-		<limit lower="-2.35619449" upper="1.30899694" effort="10" velocity="2"/>
+		<limit lower="-2.35619449" upper="1.30899694" effort="6.0" velocity="6.597344565"/>
 	</joint>
 	<joint name="RShoulderRoll" type="revolute">
@@ -47,5 +48,5 @@
 		<origin xyz="0.002 -0.03 -0.03" rpy="-0.174532925 0 0"/>
 		<axis xyz="1 0 0"/>
-		<limit lower="-1.30899694" upper="2.35619449" effort="10" velocity="2"/>
+		<limit lower="-1.30899694" upper="2.35619449" effort="6.0" velocity="6.597344565"/>
 	</joint>
 </robot>

File: hros5_description/urdf/modules/head.xacro (robot description, xacro)
@@ -1,5 +1,5 @@
 <?xml version="1.0"?>
 <robot xmlns:xacro="http://www.ros.org/wiki/xacro">
-	<joint name="HeadYaw" type="continuous">
+	<joint name="HeadYaw" type="revolute">
 		<parent link="base_link"/>
 		<child link="LowerHead"/>
@@ -7,5 +7,5 @@
 		<origin xyz="0.0035 0 0.1115" rpy="0 0 0"/>
 		<axis xyz="0 0 1"/>
-		<!-- <limit lower="-1.22173048" upper="1.22173048" effort="10" velocity="2"/> -->
+		<limit lower="-1.22173048" upper="1.22173048" effort="2.5" velocity="5.759586525"/>
 	</joint>
 	<link name="LowerHead">
@@ -17,5 +17,5 @@
 		<origin xyz="-0.01 0 0.049" rpy="0 0 0"/>
 		<axis xyz="0 1 0"/>
-		<limit upper="0.4" lower="-0.25" effort="10" velocity="2"/>
+		<limit upper="0.4" lower="-0.25" effort="2.5" velocity="5.759586525"/>
 	</joint>
 	<link name="UpperHeadBase">

File: hros5_description/urdf/modules/legs.xacro (robot description, xacro)
@@ -8,5 +8,5 @@
 			<origin xyz="0.0175 ${reflect*0.048} -0.063" rpy="0 0 0"/>
 			<axis xyz="0 0 1"/>
-			<limit lower="-0.523598776" upper="0.523598776" effort="10" velocity="2"/>
+			<limit lower="-0.523598776" upper="0.523598776" effort="8.4" velocity="4.712388975"/>
 		</joint>
 		<link name="${side}Hip">
@@ -19,5 +19,5 @@
 			<origin xyz="-0.0675 0 -0.034" rpy="0 0 0"/>
 			<axis xyz="1 0 0"/>
-			<limit lower="-0.785398163" upper="0.785398163" effort="10" velocity="2"/>
+			<limit lower="-0.785398163" upper="0.785398163" effort="8.4" velocity="4.712388975"/>
 		</joint>
 		<link name="${side}HipMotors">
@@ -29,5 +29,5 @@
 			<origin xyz="0.0705 0 0" rpy="0 0 0"/>
 			<axis xyz="0 1 0"/>
-			<limit lower="-1.57079633" upper="1.57079633" effort="10" velocity="2"/>
+			<limit lower="-1.57079633" upper="1.57079633" effort="8.4" velocity="4.712388975"/>
 		</joint>
 		<link name="${side}Thigh">
@@ -39,5 +39,5 @@
 			<origin xyz="0.0017 0 -0.127" rpy="0 0 0"/>
 			<axis xyz="0 1 0"/>
-			<limit lower="-2.7925268" upper="2.7925268" effort="10" velocity="2"/>
+			<limit lower="-2.7925268" upper="2.7925268" effort="8.4" velocity="4.712388975"/>
 		</joint>
 		<link name="${side}Tibia">
@@ -50,5 +50,5 @@
 			<!-- <origin xyz="0.024303 0.052837 -0.336141" rpy="0 0 0"/> -->
 			<axis xyz="0 1 0"/>
-			<limit lower="-1.57079633" upper="1.57079633" effort="10" velocity="2"/>
+			<limit lower="-1.57079633" upper="1.57079633" effort="8.4" velocity="4.712388975"/>
 		</joint>
 		<link name="${side}Ankle">
@@ -60,5 +60,5 @@
 			<origin xyz="-0.07 0 0" rpy="0 0 0"/>
 			<axis xyz="1 0 0"/>
-			<limit lower="-0.785398163" upper="0.785398163" effort="10" velocity="2"/>
+			<limit lower="-0.785398163" upper="0.785398163" effort="8.4" velocity="4.712388975"/>
 		</joint>
 		<link name="${side}Foot">

Commit message: Added links for ROS REP compatibility

File: hros5_description/urdf/modules/arms.xacro (robot description, xacro)
@@ -50,3 +50,16 @@
 		<limit lower="-1.30899694" upper="2.35619449" effort="6.0" velocity="6.597344565"/>
 	</joint>
+<!-- ROS REP LINKS -->
+	<joint name="l_wrist_joint" type="fixed">
+		<parent link="LLowerArm"/>
+		<child link="l_wrist"/>
+		<origin xyz="0 0 -0.0425" rpy="0 0 0"/>
+	</joint>
+	<link name="l_wrist"/>
+	<joint name="r_wrist_joint" type="fixed">
+		<parent link="RLowerArm"/>
+		<child link="r_wrist"/>
+		<origin xyz="0 0 -0.0425" rpy="0 0 0"/>
+	</joint>
+	<link name="r_wrist"/>
 </robot>

File: hros5_description/urdf/modules/head.xacro (robot description, xacro)
@@ -43,3 +43,10 @@
 		<xacro:visuals_collisions_upper_head_back/>
 	</link>
+<!-- ROS REP LINKS -->
+	<joint name="gaze_joint" type="fixed">
+		<parent link="UpperHeadBase"/>
+		<child link="gaze"/>
+		<origin xyz="0 0 0" rpy="0 0 0"/>
+	</joint>
+	<link name="gaze"/>
 </robot>

File: hros5_description/urdf/modules/legs.xacro (robot description, xacro)
@@ -68,3 +68,28 @@
 	<xacro:legs_links_joints reflect="1" side="L"/>
 	<xacro:legs_links_joints reflect="-1" side="R"/>
+<!-- ROS REP LINKS -->
+	<joint name="l_ankle_joint" type="fixed">
+		<parent link="LAnkle"/>
+		<child link="l_ankle"/>
+		<origin xyz="0 0 0" rpy="0 0 0"/>
+	</joint>
+	<link name="l_ankle"/>
+	<joint name="r_ankle_joint" type="fixed">
+		<parent link="RAnkle"/>
+		<child link="r_ankle"/>
+		<origin xyz="0 0 0" rpy="0 0 0"/>
+	</joint>
+	<link name="r_ankle"/>
+	<joint name="l_sole_joint" type="fixed">
+		<parent link="LFoot"/>
+		<child link="l_sole"/>
+		<origin xyz="0.0565 0.007 -0.04" rpy="0 0 0"/>
+	</joint>
+	<link name="l_sole"/>
+	<joint name="r_sole_joint" type="fixed">
+		<parent link="RFoot"/>
+		<child link="r_sole"/>
+		<origin xyz="0.0565 -0.007 -0.04" rpy="0 0 0"/>
+	</joint>
+	<link name="r_sole"/>
 </robot>

Commit message: First attempt to add MoveIt! integration..Seems OK!

File: hros5_description/urdf/modules/arms.xacro (robot description, xacro)
@@ -3,5 +3,5 @@
 	<xacro:macro name="arms_links_joints" params="side reflect">
 		<joint name="${side}ShoulderPitch" type="revolute">
-			<parent link="base_link"/>
+			<parent link="torso"/>
 			<child link="${side}Shoulder"/>
 			<!-- <origin xyz="-0.001114 0.079433 0.072086" rpy="0 0 0"/> -->
@@ -23,11 +23,4 @@
 			<xacro:visuals_collisions_upper_arm side="${side}" reflect="${reflect}"/>
 		</link>
-		<joint name="${side}ElbowPitch" type="revolute">
-			<parent link="${side}UpperArm"/>
-			<child link="${side}LowerArm"/>
-			<origin xyz="0.03 ${reflect*-0.0015} -0.085" rpy="0 0 0"/>
-			<axis xyz="0 1 0"/>
-			<limit lower="${reflect*-1.22173048}" upper="${reflect*1.65806279}" effort="6.0" velocity="6.597344565"/>
-		</joint>
 		<link name="${side}LowerArm">
 			<xacro:visuals_collisions_lower_arm side="${side}" reflect="${reflect}"/>
@@ -50,4 +43,18 @@
 		<limit lower="-1.30899694" upper="2.35619449" effort="6.0" velocity="6.597344565"/>
 	</joint>
+	<joint name="LElbowPitch" type="revolute">
+		<parent link="LUpperArm"/>
+		<child link="LLowerArm"/>
+		<origin xyz="0.03 -0.0015 -0.085" rpy="0 0 0"/>
+		<axis xyz="0 1 0"/>
+		<limit lower="-1.22173048" upper="1.65806279" effort="6.0" velocity="6.597344565"/>
+	</joint>
+	<joint name="RElbowPitch" type="revolute">
+		<parent link="RUpperArm"/>
+		<child link="RLowerArm"/>
+		<origin xyz="0.03 0.0015 -0.085" rpy="0 0 0"/>
+		<axis xyz="0 1 0"/>
+		<limit lower="-1.65806279" upper="1.22173048" effort="6.0" velocity="6.597344565"/>
+	</joint>
 <!-- ROS REP LINKS -->
 	<joint name="l_wrist_joint" type="fixed">

File: hros5_description/urdf/modules/head.xacro (robot description, xacro)
@@ -2,5 +2,5 @@
 <robot xmlns:xacro="http://www.ros.org/wiki/xacro">
 	<joint name="HeadYaw" type="revolute">
-		<parent link="base_link"/>
+		<parent link="torso"/>
 		<child link="LowerHead"/>
 		<!-- <origin xyz="-0.00661 -0.014699 0.16054" rpy="0 0 0"/> -->

File: hros5_description/urdf/modules/legs.xacro (robot description, xacro)
@@ -3,5 +3,5 @@
 	<xacro:macro name="legs_links_joints" params="side reflect">
 		<joint name="${side}HipYaw" type="revolute">
-			<parent link="base_link"/>
+			<parent link="torso"/>
 			<child link="${side}Hip"/>
 			<!-- <origin xyz="-0.00145 0.048 -0.071931" rpy="0 0 0"/> -->
