Commit message: Added limits and fixed 3d models error

File: hros5_description/urdf/hros5_visuals_collisions_endoskeleton.xacro (robot description, xacro)
@@ -203,5 +203,5 @@
 	<xacro:macro name="visuals_collisions_foot" params="side">
 		<visual>
-			<origin xyz="0.065 ${reflect*0.007} -0.026" rpy="0 0 0"/>
+			<origin xyz="0.0565 ${reflect*0.007} -0.031" rpy="0 0 0"/>
 			<geometry>
 				<mesh filename="package://hros5_description/meshes/endoskeleton/visual/${side}Foot.dae" scale="${scale} ${scale} ${scale}"/>
@@ -209,5 +209,5 @@
 		</visual>
 		<collision>
-			<origin xyz="0.065 ${reflect*0.007} -0.026" rpy="0 0 0"/>
+			<origin xyz="0.0565 ${reflect*0.007} -0.031" rpy="0 0 0"/>
 			<geometry>
 				<mesh filename="package://hros5_description/meshes/endoskeleton/collision/${side}Foot.stl" scale="${scale} ${scale} ${scale}"/>

File: hros5_description/urdf/modules/arms.xacro (robot description, xacro)
@@ -12,18 +12,20 @@
 			<xacro:visuals_collisions_shoulder side="${side}" reflect="${reflect}"/>
 		</link>
-		<joint name="${side}ShoulderRoll" type="continuous">
+		<joint name="${side}ShoulderRoll" type="revolute">
 			<parent link="${side}Shoulder"/>
 			<child link="${side}UpperArm"/>
 			<origin xyz="0.002 ${reflect*0.03} -0.03" rpy="${reflect*0.174532925} 0 0"/>
 			<axis xyz="1 0 0"/>
+			<limit lower="${reflect*-2.35619449}" upper="${reflect*1.30899694}" effort="10" velocity="2"/>
 		</joint>
 		<link name="${side}UpperArm">
 			<xacro:visuals_collisions_upper_arm side="${side}" reflect="${reflect}"/>
 		</link>
-		<joint name="${side}ElbowPitch" type="continuous">
+		<joint name="${side}ElbowPitch" type="revolute">
 			<parent link="${side}UpperArm"/>
 			<child link="${side}LowerArm"/>
 			<origin xyz="0.03 ${reflect*-0.0015} -0.085" rpy="0 0 0"/>
 			<axis xyz="0 1 0"/>
+			<limit lower="${reflect*-1.22173048}" upper="${reflect*1.65806279}" effort="10" velocity="2"/>
 		</joint>
 		<link name="${side}LowerArm">

File: hros5_description/urdf/modules/head.xacro (robot description, xacro)
@@ -7,4 +7,5 @@
 		<origin xyz="0.0035 0 0.1115" rpy="0 0 0"/>
 		<axis xyz="0 0 1"/>
+		<!-- <limit lower="-1.22173048" upper="1.22173048" effort="10" velocity="2"/> -->
 	</joint>
 	<link name="LowerHead">

File: hros5_description/urdf/modules/legs.xacro (robot description, xacro)
@@ -2,5 +2,5 @@
 <robot xmlns:xacro="http://www.ros.org/wiki/xacro">
 	<xacro:macro name="legs_links_joints" params="side reflect">
-		<joint name="${side}HipYaw" type="continuous">
+		<joint name="${side}HipYaw" type="revolute">
 			<parent link="base_link"/>
 			<child link="${side}Hip"/>
@@ -8,9 +8,10 @@
 			<origin xyz="0.0175 ${reflect*0.048} -0.063" rpy="0 0 0"/>
 			<axis xyz="0 0 1"/>
+			<limit lower="-0.523598776" upper="0.523598776" effort="10" velocity="2"/>
 		</joint>
 		<link name="${side}Hip">
 			<xacro:visuals_collisions_hip side="${side}"/>
 		</link>
-		<joint name="${side}HipRoll" type="continuous">
+		<joint name="${side}HipRoll" type="revolute">
 			<parent link="${side}Hip"/>
 			<child link="${side}HipMotors"/>
@@ -18,27 +19,30 @@
 			<origin xyz="-0.0675 0 -0.034" rpy="0 0 0"/>
 			<axis xyz="1 0 0"/>
+			<limit lower="-0.785398163" upper="0.785398163" effort="10" velocity="2"/>
 		</joint>
 		<link name="${side}HipMotors">
 			<xacro:visuals_collisions_hip_motors side="${side}"/>
 		</link>
-		<joint name="${side}HipPitch" type="continuous">
+		<joint name="${side}HipPitch" type="revolute">
 			<parent link="${side}HipMotors"/>
 			<child link="${side}Thigh"/>
 			<origin xyz="0.0705 0 0" rpy="0 0 0"/>
 			<axis xyz="0 1 0"/>
+			<limit lower="-1.57079633" upper="1.57079633" effort="10" velocity="2"/>
 		</joint>
 		<link name="${side}Thigh">
 			<xacro:visuals_collisions_thigh side="${side}"/>
 		</link>
-		<joint name="${side}KneePitch" type="continuous">
+		<joint name="${side}KneePitch" type="revolute">
 			<parent link="${side}Thigh"/>
 			<child link="${side}Tibia"/>
 			<origin xyz="0.0017 0 -0.127" rpy="0 0 0"/>
 			<axis xyz="0 1 0"/>
+			<limit lower="-2.7925268" upper="2.7925268" effort="10" velocity="2"/>
 		</joint>
 		<link name="${side}Tibia">
 			<xacro:visuals_collisions_tibia side="${side}"/>
 		</link>
-		<joint name="${side}AnklePitch" type="continuous">
+		<joint name="${side}AnklePitch" type="revolute">
 			<parent link="${side}Tibia"/>
 			<child link="${side}Ankle"/>
@@ -46,13 +50,15 @@
 			<!-- <origin xyz="0.024303 0.052837 -0.336141" rpy="0 0 0"/> -->
 			<axis xyz="0 1 0"/>
+			<limit lower="-1.57079633" upper="1.57079633" effort="10" velocity="2"/>
 		</joint>
 		<link name="${side}Ankle">
 			<xacro:visuals_collisions_ankle side="${side}"/>
 		</link>
-		<joint name="${side}AnkleRoll" type="continuous">
+		<joint name="${side}AnkleRoll" type="revolute">
 			<parent link="${side}Ankle"/>
 			<child link="${side}Foot"/>
 			<origin xyz="-0.07 0 0" rpy="0 0 0"/>
 			<axis xyz="1 0 0"/>
+			<limit lower="-0.785398163" upper="0.785398163" effort="10" velocity="2"/>
 		</joint>
 		<link name="${side}Foot">

Commit message: Small fix in meshes/URDF

File: hros5_description/urdf/hros5_visuals_collisions_endoskeleton.xacro (robot description, xacro)
@@ -95,5 +95,5 @@
 	<xacro:macro name="visuals_collisions_upper_arm" params="side reflect">
 		<visual>
-			<origin xyz="0 ${reflect*-0.00025} -0.0395" rpy="0 0 0"/>
+			<origin xyz="0 -0.0005 -0.0395" rpy="0 0 0"/>
 			<geometry>
 				<mesh filename="package://hros5_description/meshes/endoskeleton/visual/${side}UpperArm.dae" scale="${scale} ${scale} ${scale}"/>
@@ -128,5 +128,5 @@
 			<origin xyz="-0.01605 0 -0.008931" rpy="0 0 0"/>
 			<geometry>
-				<mesh filename="package://hros5_description/meshes/endoskeleton/visual/${side}Hip.dae" scale="${scale} ${scale} ${scale}"/>
+				<mesh filename="package://hros5_description/meshes/endoskeleton/visual/Hip.dae" scale="${scale} ${scale} ${scale}"/>
 			</geometry>
 		</visual>
@@ -134,5 +134,5 @@
 			<origin xyz="-0.01605 0 -0.008931" rpy="0 0 0"/>
 			<geometry>
-				<mesh filename="package://hros5_description/meshes/endoskeleton/collision/${side}Hip.stl" scale="${scale} ${scale} ${scale}"/>
+				<mesh filename="package://hros5_description/meshes/endoskeleton/collision/Hip.stl" scale="${scale} ${scale} ${scale}"/>
 			</geometry>
 		</collision>
@@ -143,5 +143,5 @@
 			<origin xyz="0.077 -0.0052 -0.0041" rpy="0 0 0"/>
 			<geometry>
-				<mesh filename="package://hros5_description/meshes/endoskeleton/visual/${side}HipMotors.dae" scale="${scale} ${scale} ${scale}"/>
+				<mesh filename="package://hros5_description/meshes/endoskeleton/visual/HipMotors.dae" scale="${scale} ${scale} ${scale}"/>
 			</geometry>
 		</visual>
@@ -149,5 +149,5 @@
 			<origin xyz="0.077 -0.0052 -0.0041" rpy="0 0 0"/>
 			<geometry>
-				<mesh filename="package://hros5_description/meshes/endoskeleton/collision/${side}HipMotors.stl" scale="${scale} ${scale} ${scale}"/>
+				<mesh filename="package://hros5_description/meshes/endoskeleton/collision/HipMotors.stl" scale="${scale} ${scale} ${scale}"/>
 			</geometry>
 		</collision>
@@ -159,5 +159,5 @@
 			<origin xyz="0.001 -0.0095 -0.095" rpy="0 0 0"/>
 			<geometry>
-				<mesh filename="package://hros5_description/meshes/endoskeleton/visual/${side}Thigh.dae" scale="${scale} ${scale} ${scale}"/>
+				<mesh filename="package://hros5_description/meshes/endoskeleton/visual/Thigh.dae" scale="${scale} ${scale} ${scale}"/>
 			</geometry>
 		</visual>
@@ -165,5 +165,5 @@
 			<origin xyz="0.001 -0.0095 -0.095" rpy="0 0 0"/>
 			<geometry>
-				<mesh filename="package://hros5_description/meshes/endoskeleton/collision/${side}Thigh.stl" scale="${scale} ${scale} ${scale}"/>
+				<mesh filename="package://hros5_description/meshes/endoskeleton/collision/Thigh.stl" scale="${scale} ${scale} ${scale}"/>
 			</geometry>
 		</collision>
@@ -175,5 +175,5 @@
 			<origin xyz="0.004 0 -0.059" rpy="0 0 0"/>
 			<geometry>
-				<mesh filename="package://hros5_description/meshes/endoskeleton/visual/${side}Tibia.dae" scale="${scale} ${scale} ${scale}"/>
+				<mesh filename="package://hros5_description/meshes/endoskeleton/visual/Tibia.dae" scale="${scale} ${scale} ${scale}"/>
 			</geometry>
 		</visual>
@@ -181,5 +181,5 @@
 			<origin xyz="0.004 0 -0.059" rpy="0 0 0"/>
 			<geometry>
-				<mesh filename="package://hros5_description/meshes/endoskeleton/collision/${side}Tibia.stl" scale="${scale} ${scale} ${scale}"/>
+				<mesh filename="package://hros5_description/meshes/endoskeleton/collision/Tibia.stl" scale="${scale} ${scale} ${scale}"/>
 			</geometry>
 		</collision>
@@ -190,5 +190,5 @@
 			<origin xyz="0.00625 0.00525 0.0042" rpy="0 0 0"/>
 			<geometry>
-				<mesh filename="package://hros5_description/meshes/endoskeleton/visual/${side}Ankle.dae" scale="${scale} ${scale} ${scale}"/>
+				<mesh filename="package://hros5_description/meshes/endoskeleton/visual/Ankle.dae" scale="${scale} ${scale} ${scale}"/>
 			</geometry>
 		</visual>
@@ -196,5 +196,5 @@
 			<origin xyz="0.00625 0.00525 0.0042" rpy="0 0 0"/>
 			<geometry>
-				<mesh filename="package://hros5_description/meshes/endoskeleton/collision/${side}Ankle.stl" scale="${scale} ${scale} ${scale}"/>
+				<mesh filename="package://hros5_description/meshes/endoskeleton/collision/Ankle.stl" scale="${scale} ${scale} ${scale}"/>
 			</geometry>
 		</collision>

File: hros5_description/urdf/modules/arms.xacro (robot description, xacro)
@@ -53,5 +53,5 @@
 		<parent link="RUpperArm"/>
 		<child link="RLowerArm"/>
-		<origin xyz="0.03 0.0015 -0.085" rpy="0 0 0"/>
+		<origin xyz="0.03 -0.0015 -0.085" rpy="0 0 0"/>
 		<axis xyz="0 1 0"/>
 		<limit lower="-1.65806279" upper="1.22173048" effort="6.0" velocity="6.597344565"/>

Commit message: Small fix in meshes/URDF

File: hros5_description/urdf/hros5_visuals_collisions_endoskeleton.xacro (robot description, xacro)
@@ -110,5 +110,5 @@
 	<xacro:macro name="visuals_collisions_lower_arm" params="side reflect">
 		<visual>
-			<origin xyz="-0.0023 0 -0.0408" rpy="0 0 0"/>
+			<origin xyz="0 ${reflect*-0.003} -0.0204" rpy="0 0 0"/>
 			<geometry>
 				<mesh filename="package://hros5_description/meshes/endoskeleton/visual/${side}LowerArm.dae" scale="${scale} ${scale} ${scale}"/>
@@ -116,5 +116,5 @@
 		</visual>
 		<collision>
-			<origin xyz="-0.0023 0 -0.0408" rpy="0 0 0"/>
+			<origin xyz="0 ${reflect*-0.003} -0.0204" rpy="0 0 0"/>
 			<geometry>
 				<mesh filename="package://hros5_description/meshes/endoskeleton/collision/${side}LowerArm.stl" scale="${scale} ${scale} ${scale}"/>

Commit message: Dummy inertia from Darwin OP and fixes for first simple Gazebo Simulation

File: hros5_description/urdf/hros5_visuals_collisions_endoskeleton.xacro (robot description, xacro)
@@ -35,5 +35,4 @@
 	<xacro:macro name="visuals_collisions_upper_head_base" params="">
 		<visual>
-			<!-- <origin xyz="-0.01175 -0.0025 0.033" rpy="0 0 0"/> -->
 			<origin xyz="0.0075 -0.0045 0.0275" rpy="0 0 0"/>
 			<geometry>
@@ -156,5 +155,4 @@
 	<xacro:macro name="visuals_collisions_thigh" params="side">
 		<visual>
-			<!-- <origin xyz="0.043764 0.038393 -0.188164" rpy="0 0 0"/> -->
 			<origin xyz="0.001 -0.0095 -0.095" rpy="0 0 0"/>
 			<geometry>
@@ -172,5 +170,4 @@
 	<xacro:macro name="visuals_collisions_tibia" params="side">
 		<visual>
-			<!-- <origin xyz="0.041317 0.047709 -0.276974" rpy="0 0 0"/> -->
 			<origin xyz="0.004 0 -0.059" rpy="0 0 0"/>
 			<geometry>

File: hros5_description/urdf/modules/arms.xacro (robot description, xacro)
@@ -5,5 +5,4 @@
 			<parent link="torso"/>
 			<child link="${side}Shoulder"/>
-			<!-- <origin xyz="-0.001114 0.079433 0.072086" rpy="0 0 0"/> -->
 			<origin xyz="0.003 ${reflect*0.0675} 0.084" rpy="0 0 0"/>
 			<axis xyz="0 1 0"/>
@@ -12,17 +11,25 @@
 		<link name="${side}Shoulder">
 			<xacro:visuals_collisions_shoulder side="${side}" reflect="${reflect}"/>
+			<inertial> <!-- Dummy values from Darwin OP -->
+				<origin xyz="-0.013522619 0.010264050 0.0013935747" />
+				<mass value="0.025913024"/>
+				<inertia ixx="0.0097758165"  ixy="0.0016911839"  ixz="-0.00045174329" iyx="0.0016911839" iyy="0.010511104" iyz="0.00033406955" izx="-0.00045174329" izy="0.00033406955" izz="0.005476798" />
+		    </inertial>
 		</link>
-		<!-- <joint name="${side}ShoulderRoll" type="revolute">
-			<parent link="${side}Shoulder"/>
-			<child link="${side}UpperArm"/>
-			<origin xyz="0.002 ${reflect*0.03} -0.03" rpy="${reflect*0.174532925} 0 0"/>
-			<axis xyz="1 0 0"/>
-			<limit lower="${reflect*-2.35619449}" upper="${reflect*1.30899694}" effort="6.0" velocity="6.597344565"/>
-		</joint> -->
 		<link name="${side}UpperArm">
 			<xacro:visuals_collisions_upper_arm side="${side}" reflect="${reflect}"/>
+			<inertial> <!-- Dummy values from Darwin OP -->
+				<origin xyz="-0.036239 0.000734 0.000660" />
+				<mass value="0.16837715"/>
+				<inertia ixx="0.12202839"  ixy="-0.0020812626"  ixz="-0.00088143449" iyx="-0.0020812626" iyy="0.038088441" iyz="0.0018251448" izx="-0.00088143449" izy="0.0018251448" izz="0.11340830" />
+		    </inertial>
 		</link>
 		<link name="${side}LowerArm">
 			<xacro:visuals_collisions_lower_arm side="${side}" reflect="${reflect}"/>
+			<inertial> <!-- Dummy values from Darwin OP -->
+				<origin xyz="0.000000 0.000000 0.000000"/>
+				<mass value="0.059288504"/>
+				<inertia ixx="0.086855267"  ixy="0.0053020311"  ixz="0.00043636051" iyx="0.0053020311" iyy="0.021192085" iyz="-0.0064855932" izx="0.00043636051" izy="-0.0064855932" izz="0.086845450" />
+		    </inertial>
 		</link>
 	</xacro:macro>

File: hros5_description/urdf/modules/head.xacro (robot description, xacro)
@@ -4,5 +4,4 @@
 		<parent link="torso"/>
 		<child link="LowerHead"/>
-		<!-- <origin xyz="-0.00661 -0.014699 0.16054" rpy="0 0 0"/> -->
 		<origin xyz="0.0035 0 0.1115" rpy="0 0 0"/>
 		<axis xyz="0 0 1"/>
@@ -11,4 +10,9 @@
 	<link name="LowerHead">
 		<xacro:visuals_collisions_lower_head/>
+		<inertial> <!-- Dummy values from Darwin OP -->
+			<origin xyz="0.001424 -0.016567 -0.007128" />
+			<mass value="0.024357719"/>
+			<inertia ixx="0.0051411124"  ixy="-0.00057530255"  ixz="-0.000024729049" iyy="0.0081915737" iyz="-0.000019223094" izz="0.0011379812" />
+	    </inertial>
 	</link>
 	<joint name="HeadPitch" type="revolute">
@@ -21,4 +25,9 @@
 	<link name="UpperHeadBase">
 		<xacro:visuals_collisions_upper_head_base/>
+		<inertial> <!-- Dummy values from Darwin OP -->
+			<origin xyz="0.000064 -0.018565 -0.007667" />
+			<mass value="0.15804192"/>
+			<inertia ixx="0.1239683"  ixy="0.000078494368"  ixz="0.000007645979" iyy="0.11783781" iyz="0.0012199205" izz="0.1583601" />
+	    </inertial>
 	</link>
 	<joint name="HeadPitchDummy" type="continuous">
@@ -35,5 +44,4 @@
 		<parent link="LowerHead"/>
 		<child link="UpperHeadBack"/>
-		<!-- <origin xyz="-0.04 0 -0.074" rpy="0 0 0"/> -->
 		<origin xyz="-0.0525 0 0.021" rpy="0 0 0"/>
 		<axis xyz="0 1 0"/>

File: hros5_description/urdf/modules/legs.xacro (robot description, xacro)
@@ -5,5 +5,4 @@
 			<parent link="torso"/>
 			<child link="${side}Hip"/>
-			<!-- <origin xyz="-0.00145 0.048 -0.071931" rpy="0 0 0"/> -->
 			<origin xyz="0.0175 ${reflect*0.048} -0.063" rpy="0 0 0"/>
 			<axis xyz="0 0 1"/>
@@ -12,9 +11,13 @@
 		<link name="${side}Hip">
 			<xacro:visuals_collisions_hip side="${side}"/>
+			<inertial> <!-- Dummy values from Darwin OP -->
+				<origin xyz="0.000000 0.000480 0.018437" />
+				<mass value="0.167"/>
+				<inertia ixx="0.12259691"  ixy="0.00071127469"  ixz="0.00081143913" iyx="0.00071127469" iyy="0.11066637" iyz="-0.0071635476" izx="0.00081143913" izy="-0.0071635476" izz="0.041877668" />
+			</inertial>
 		</link>
 		<joint name="${side}HipRoll" type="revolute">
 			<parent link="${side}Hip"/>
 			<child link="${side}HipMotors"/>
-			<!-- <origin xyz="0.047519 0.048 -0.097025" rpy="0 0 0"/> 0.0033019-->
 			<origin xyz="-0.0675 0 -0.034" rpy="0 0 0"/>
 			<axis xyz="1 0 0"/>
@@ -23,4 +26,9 @@
 		<link name="${side}HipMotors">
 			<xacro:visuals_collisions_hip_motors side="${side}"/>
+			<inertial> <!-- Dummy values from Darwin OP -->
+				<origin xyz="0.000000 0.000480 0.018437" />
+				<mass value="0.167"/>
+				<inertia ixx="0.12259691"  ixy="0.00071127469"  ixz="0.00081143913" iyx="0.00071127469" iyy="0.11066637" iyz="-0.0071635476" izx="0.00081143913" izy="-0.0071635476" izz="0.041877668" />
+			</inertial>
 		</link>
 		<joint name="${side}HipPitch" type="revolute">
@@ -33,4 +41,9 @@
 		<link name="${side}Thigh">
 			<xacro:visuals_collisions_thigh side="${side}"/>
+			<inertial> <!-- Dummy values from Darwin OP -->
+				<origin xyz="0.000079 0.018242 0.013873" />
+				<mass value="0.11904336"/>
+				<inertia ixx="0.097950272"  ixy="0.0012119368"  ixz="-0.00021223016" iyx="0.00122119368" iyy="0.032848287" iyz="-0.0019474021" izx="-0.00021223016" izy="-0.0019474021" izz="0.11493509" />
+			</inertial>
 		</link>
 		<joint name="${side}KneePitch" type="revolute">
@@ -43,4 +56,9 @@
 		<link name="${side}Tibia">
 			<xacro:visuals_collisions_tibia side="${side}"/>
+			<inertial> <!-- Dummy values from Darwin OP -->
+				<origin xyz="-0.053955 0.006548 -0.000592" />
+				<mass value="0.070309794"/>
+				<inertia ixx="0.093369608"  ixy="-0.00093567395"  ixz="-0.00023992085" iyx="-0.00093567395" iyy="0.046295534" iyz="-0.012858493" izx="-0.00023992085" izy="-0.012858493" izz="0.11351516" />
+			</inertial>
 		</link>
 		<joint name="${side}AnklePitch" type="revolute">
@@ -48,5 +66,4 @@
 			<child link="${side}Ankle"/>
 			<origin xyz="-0.002 0 -0.125" rpy="0 0 0"/>
-			<!-- <origin xyz="0.024303 0.052837 -0.336141" rpy="0 0 0"/> -->
 			<axis xyz="0 1 0"/>
 			<limit lower="-1.57079633" upper="1.57079633" effort="8.4" velocity="4.712388975"/>
@@ -54,4 +71,9 @@
 		<link name="${side}Ankle">
 			<xacro:visuals_collisions_ankle side="${side}"/>
+			<inertial> <!-- Dummy values from Darwin OP -->
+				<origin xyz="-0.000214 -0.018536 0.013873" />
+				<mass value="0.16710792"/>
+				<inertia ixx="0.12079175"  ixy="-0.00079781067"  ixz="-0.00039322246" iyx="-0.00079781067" iyy="0.10885465" iyz="0.0070770117" izx="-0.00039322246" izy="0.0070770117" izz="0.041871103" />
+			</inertial>
 		</link>
 		<joint name="${side}AnkleRoll" type="revolute">
@@ -64,4 +86,9 @@
 		<link name="${side}Foot">
 			<xacro:visuals_collisions_foot side="${side}"/>
+			<inertial> <!-- Dummy values from Darwin OP -->
+				<origin xyz="-0.025995 -0.009506 -0.000503" />
+				<mass value="0.0794462"/>
+				<inertia ixx="0.12079175"  ixy="-0.00079781067"  ixz="-0.00039322246" iyx="-0.00079781067" iyy="0.10885465" iyz="0.0070770117" izx="-0.00039322246" izy="0.0070770117" izz="0.041871103" />
+			</inertial>
 		</link>
 	</xacro:macro>

File: hros5_description/urdf/modules/torso.xacro (robot description, xacro)
@@ -10,4 +10,9 @@
 	<link name="torso">
 		<xacro:visuals_collisions_torso/>
+		<inertial> <!-- Dummy values from Darwin OP -->
+			<origin xyz="-0.003053 -0.038651 -0.019268" />
+			<mass value="0.97559947"/>
+			<inertia ixx="3.1081800"  ixy="-0.25460189"  ixz="2.0318174" iyy="6.3787776" iyz="0.16417863" izz="5.3316425" />
+		</inertial>
 	</link>
 </robot>
