Commit message: Additions to Gazebo URDF

File: hros5_description/urdf/hros5.urdf (robot description, URDF)
Before this commit: robot hros5, 31 links, 30 joints
Links:
- link LAnkle: mass None -> 0.16710792; geometry collision mesh filename=package://hros5_description/meshes/endoskeleton/collision/A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 scale=0.1 0.1 0.1; visual mesh filename=package://hros5_description/meshes/endoskeleton/visual/Ankl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 scale=0.1 0.1 0.1
- link LFoot: mass None -> 0.0794462
- link LHip: mass None -> 0.167; geometry collision mesh filename=package://hros5_description/meshes/endoskeleton/collision/H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 scale=0.1 0.1 0.1; visual mesh filename=package://hros5_description/meshes/endoskeleton/visual/Hip.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 scale=0.1 0.1 0.1
- link LHipMotors: mass None -> 0.167; geometry collision mesh filename=package://hros5_description/meshes/endoskeleton/collision/H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 scale=0.1 0.1 0.1; visual mesh filename=package://hros5_description/meshes/endoskeleton/visual/HipM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 scale=0.1 0.1 0.1
- link LLowerArm: mass None -> 0.059288504
- link LShoulder: mass None -> 0.025913024
- link LThigh: mass None -> 0.11904336; geometry collision mesh filename=package://hros5_description/meshes/endoskeleton/collision/T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 scale=0.1 0.1 0.1; visual mesh filename=package://hros5_description/meshes/endoskeleton/visual/Thig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 scale=0.1 0.1 0.1
- link LTibia: mass None -> 0.070309794; geometry collision mesh filename=package://hros5_description/meshes/endoskeleton/collision/T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 scale=0.1 0.1 0.1; visual mesh filename=package://hros5_description/meshes/endoskeleton/visual/Tibi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 scale=0.1 0.1 0.1
- link LUpperArm: mass None -> 0.16837715
- link LowerHead: mass None -> 0.024357719
- link RAnkle: mass None -> 0.16710792; geometry collision mesh filename=package://hros5_description/meshes/endoskeleton/collision/A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 scale=0.1 0.1 0.1; visual mesh filename=package://hros5_description/meshes/endoskeleton/visual/Ankl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 scale=0.1 0.1 0.1
- link RFoot: mass None -> 0.0794462
- link RHip: mass None -> 0.167; geometry collision mesh filename=package://hros5_description/meshes/endoskeleton/collision/H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 scale=0.1 0.1 0.1; visual mesh filename=package://hros5_description/meshes/endoskeleton/visual/Hip.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 scale=0.1 0.1 0.1
- link RHipMotors: mass None -> 0.167; geometry collision mesh filename=package://hros5_description/meshes/endoskeleton/collision/H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 scale=0.1 0.1 0.1; visual mesh filename=package://hros5_description/meshes/endoskeleton/visual/HipM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 scale=0.1 0.1 0.1
- link RLowerArm: mass None -> 0.059288504
- link RShoulder: mass None -> 0.025913024
- link RThigh: mass None -> 0.11904336; geometry collision mesh filename=package://hros5_description/meshes/endoskeleton/collision/T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 scale=0.1 0.1 0.1; visual mesh filename=package://hros5_description/meshes/endoskeleton/visual/Thig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 scale=0.1 0.1 0.1
- link RTibia: mass None -> 0.070309794; geometry collision mesh filename=package://hros5_description/meshes/endoskeleton/collision/T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 scale=0.1 0.1 0.1; visual mesh filename=package://hros5_description/meshes/endoskeleton/visual/Tibi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 scale=0.1 0.1 0.1
- link RUpperArm: mass None -> 0.16837715
- link UpperHeadBack: mass None -> 0.2e-5
- link UpperHeadBase: mass None -> 0.15804192
- link UpperHeadMotor: mass None -> 0.2e-5
- link torso: mass None -> 0.97559947
Joints:
- joint RElbowPitch: origin xyz=0.03 0.0015 -0.085 rpy=0 0 0 -> xyz=0.03 -0.0015 -0.085 rpy=0 0 0

File: hros5_description/urdf/hros5_gazebo.xacro (robot description, xacro)
@@ -9,3 +9,19 @@
     </gazebo>
 <!-- END OF GAZEBO ROS CONTROL PLUGIN -->
+<!-- MIMIC JOINTS  -->
+	<gazebo>
+		<plugin name="HeadPitchDummy" filename="libroboticsgroup_gazebo_mimic_joint_plugin.so">
+			<joint>HeadPitch</joint>
+			<mimicJoint>HeadPitchDummy</mimicJoint>
+			<multiplier>-1.0</multiplier>
+			<offset>0.0</offset>
+		</plugin>
+		<plugin name="HeadPitchDummy2" filename="libroboticsgroup_gazebo_mimic_joint_plugin.so">
+			<joint>HeadPitch</joint>
+			<mimicJoint>HeadPitchDummy2</mimicJoint>
+			<multiplier>0.65</multiplier>
+			<offset>0.0</offset>
+		</plugin>
+	</gazebo>
+<!-- END OF MIMIC JOINTS -->
 </robot>

File: hros5_description/urdf/modules/head.xacro (robot description, xacro)
@@ -40,4 +40,9 @@
 	<link name="UpperHeadMotor">
 		<xacro:visuals_collisions_upper_head_motor/>
+		<inertial> <!-- dummy values for gazebo -->
+			<mass value="0.2e-5" />
+			<origin xyz="0 0 0"/>
+			<inertia ixx="1e-9" ixy="0" ixz="0" iyy="1e-9" iyz="0" izz="1e-9" />
+		</inertial>
 	</link>
 	<joint name="HeadPitchDummy2" type="continuous">
@@ -50,4 +55,9 @@
 	<link name="UpperHeadBack">
 		<xacro:visuals_collisions_upper_head_back/>
+		<inertial> <!-- dummy values for gazebo -->
+			<mass value="0.2e-5" />
+			<origin xyz="0 0 0"/>
+			<inertia ixx="1e-9" ixy="0" ixz="0" iyy="1e-9" iyz="0" izz="1e-9" />
+		</inertial>
 	</link>
 <!-- ROS REP LINKS -->

Commit message: Changed zero configuration

File: hros5_description/urdf/hros5.urdf (robot description, URDF)
Before this commit: robot hros5, 31 links, 30 joints
Joints:
- joint LElbowPitch: origin xyz=0.03 -0.0015 -0.085 rpy=0 0 0 -> xyz=0.03 -0.0015 -0.085 rpy=0 -0.785398163395 0
- joint LShoulderRoll: origin xyz=0.002 0.03 -0.03 rpy=0.174532925 0 0 -> xyz=0.002 0.03 -0.03 rpy=0.785398163395 0 0
- joint RElbowPitch: origin xyz=0.03 -0.0015 -0.085 rpy=0 0 0 -> xyz=0.03 -0.0015 -0.085 rpy=0 -0.785398163395 0
- joint RShoulderRoll: origin xyz=0.002 -0.03 -0.03 rpy=-0.174532925 0 0 -> xyz=0.002 -0.03 -0.03 rpy=-0.785398163395 0 0

File: hros5_description/urdf/modules/arms.xacro (robot description, xacro)
@@ -39,5 +39,5 @@
 		<parent link="LShoulder"/>
 		<child link="LUpperArm"/>
-		<origin xyz="0.002 0.03 -0.03" rpy="0.174532925 0 0"/>
+		<origin xyz="0.002 0.03 -0.03" rpy="${PI_2/2} 0 0"/>
 		<axis xyz="1 0 0"/>
 		<limit lower="-2.35619449" upper="1.30899694" effort="6.0" velocity="6.597344565"/>
@@ -46,5 +46,5 @@
 		<parent link="RShoulder"/>
 		<child link="RUpperArm"/>
-		<origin xyz="0.002 -0.03 -0.03" rpy="-0.174532925 0 0"/>
+		<origin xyz="0.002 -0.03 -0.03" rpy="-${PI_2/2} 0 0"/>
 		<axis xyz="1 0 0"/>
 		<limit lower="-1.30899694" upper="2.35619449" effort="6.0" velocity="6.597344565"/>
@@ -53,5 +53,5 @@
 		<parent link="LUpperArm"/>
 		<child link="LLowerArm"/>
-		<origin xyz="0.03 -0.0015 -0.085" rpy="0 0 0"/>
+		<origin xyz="0.03 -0.0015 -0.085" rpy="0 -${PI_2/2} 0"/>
 		<axis xyz="0 1 0"/>
 		<limit lower="-1.22173048" upper="1.65806279" effort="6.0" velocity="6.597344565"/>
@@ -60,5 +60,5 @@
 		<parent link="RUpperArm"/>
 		<child link="RLowerArm"/>
-		<origin xyz="0.03 -0.0015 -0.085" rpy="0 0 0"/>
+		<origin xyz="0.03 -0.0015 -0.085" rpy="0 -${PI_2/2} 0"/>
 		<axis xyz="0 1 0"/>
 		<limit lower="-1.65806279" upper="1.22173048" effort="6.0" velocity="6.597344565"/>
